File: 326pcb.kicad_pcb (KiCad board)
At the start: 2 copper layers, 50 x 50 mm, 46 parts, among them J2 OV2640Conn, J4 Conn_01x03, J6 Conn_01x03, J7 694106106102, U1 ATSAM4S8BA-AU, U2 ESP32-WROOM-32E, U3 LDL1117S30R, Y1 12MHz

Commit message: Update files, Gerbers, Drill
Parts:
- added REF**: MountingHole_3mm, MountingHole:MountingHole_3mm, F.Cu at (153.8, 47.6)
- added REF**: MountingHole_3mm, MountingHole:MountingHole_3mm, F.Cu at (196.5, 90.4)
- moved J4 7.56 mm to (184.2, 89.3)
- moved PRGM 7.56 mm to (184.2, 92.1)
- moved R4 7.55 mm to (174.9, 92.0)
- moved R9 7.55 mm to (174.9, 89.7)
- moved C14 3.68 mm to (151.4, 75.0)
- moved AP 3.68 mm to (170.7, 73.5)
- moved U2 3.67 mm to (156.5, 61.1)
- moved WS 3.59 mm to (164.2, 74.1)
- moved Net 3.59 mm to (160.2, 74.1)
- moved R8 3.54 mm to (168.5, 73.4)
- moved C10 2.88 mm to (154.7, 72.3)
- moved R6 2.88 mm to (162.2, 73.3)
- moved R7 2.88 mm to (166.2, 73.3)
- moved U3 2.20 mm to (170.1, 78.6)
- moved C12 1.96 mm to (175.7, 80.5), turned to -90 degrees
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- renumbered PROVISION to PRVSN
Routing:
- net GND: track 305.1 -> 329.6 mm
- net +3V0: track 167.3 -> 153.2 mm, vias 18 -> 14
- net SWO: track 42.7 -> 30.3 mm
- net SWDIO: track 39.5 -> 30.4 mm, vias 3 -> 1
- net MCU_TX: track 61.6 -> 55.0 mm
- net PROVISION: track 34.0 -> 40.4 mm, vias 2 -> 3
- net EN: track 87.8 -> 82.0 mm, vias 1 -> 2
- net ESP32_RX: track 32.6 -> 28.3 mm
- net Net-(U2-IO27): track 7.87 -> 4.94 mm
- net CTRL2: track 52.8 -> 54.6 mm
- net MCU_RX: track 40.5 -> 38.9 mm
- net CTRL3: track 29.6 -> 28.1 mm
- net +5V: track 29.0 -> 27.6 mm
- net MOSI: track 40.6 -> 41.6 mm
- net Net-(U2-IO26): track 4.50 -> 3.55 mm
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Other:
- board text added: "326 Webcam V1.0 2/16/26"
- board text removed: "326 Webcam V1.0"

Commit message: update pcb
Parts:
- removed JMP: JMP, Connector_PinHeader_2.54mm:PinHeader_1x02_P2.54mm_Vertical
- SW1: renamed from MCU RST
- SW2: renamed from WiFi RST
- renumbered Net to D1, WS to D2, AP to D3, PRGM to J3, USB to J5, PRVSN to SW3, IO0 to SW4
Connections:
- C3 pad 2: Net-(J1-Pin_1) -> VDD1V2
- U1 pad 8: Net-(J1-Pin_1) -> VDD1V2
Routing:
- net Net-(J1-Pin_1): track 12.4 -> 0.00 mm
- net VDD1V2: track 71.1 -> 79.7 mm
- net MOSI: track 41.6 -> 44.7 mm
- net +3V0: track 153.2 -> 154.6 mm
Other:
- board text added: "."
- board text added: "5V"
- board text added: "AP"
- board text added: "ESP RX"
- board text added: "GND"
- board text added: "IO0"
- board text added: "MCU"
- board text added: "MCU RST"
- board text added: "Net"
- board text added: "PRGM"
- board text added: "PRVSN"
- board text added: "TX"
- board text added: "WS"
- board text added: "Wifi RST"
